Commit message: Created Rviz

File: yahboom_M3Pro_description/urdf/M3Pro.urdf (robot description, URDF)
Before this commit: robot M3Pro, 20 links, 19 joints
Links:
- link arm_base_Link: geometry collision mesh filename=package://yahboom_M3Pro_description/meshes/arm_base_Link.STL; visual mesh filename=package://yahboom_M3Pro_description/meshes/arm_base_Link.STL
